Commit message: Add Go2D1 URDF

File: low-level/resources/robots/go2d1/urdf/go2d1.urdf (robot description, URDF)
Before this commit: robot go2d1_description, 21 links, 20 joints
Links:
- added link ee_gripper_link, mass 0.001
- added link gripperMover, mass 0.015046; collision mesh filename=../meshes/d1_Link07_2.dae; visual mesh filename=../meshes/d1_Link07_2.dae scale=1 1 1
- added link gripperStator, mass 0.015046; collision mesh filename=../meshes/d1_Link07_1.dae; visual mesh filename=../meshes/d1_Link07_1.dae scale=1 1 1
- added link link02, mass 0.20213; collision mesh filename=../meshes/d1_Link02.dae; visual mesh filename=../meshes/d1_Link02.dae scale=1 1 1
- added link link03, mass 0.0629; collision mesh filename=../meshes/d1_Link03.dae; visual mesh filename=../meshes/d1_Link03.dae scale=1 1 1
- added link link04, mass 0.083332; collision mesh filename=../meshes/d1_Link04.dae; visual mesh filename=../meshes/d1_Link04.dae scale=1 1 1
- added link link05, mass 0.053817; visual mesh filename=../meshes/d1_Link05.dae scale=1 1 1
- added link link06, mass 0.077892; collision mesh filename=../meshes/d1_Link06.dae; visual mesh filename=../meshes/d1_Link06.dae scale=1 1 1
- link link00: mass 0.16166 -> 0.077233
- link link01: mass 0.67332551 -> 0.13174; geometry visual mesh filename=../meshes/d1_Link01.dae scale=1 1 1
Joints:
- removed joint d1_waist
- added joint ee_gripper: type fixed, parent gripperStator, child ee_gripper_link, origin xyz=0.135 0 0 rpy=0 0 0, axis 1 0 0
- added joint z1_elbow: type revolute, parent link02, child link03, origin xyz=0 0.2693 0.0009 rpy=0 0 0, axis 0 0 -1, limit lower=-1.57 upper=1.57 effort=30.0 velocity=10
- added joint z1_forearm_roll: type revolute, parent link04, child link05, origin xyz=-0.0001 -0.0237 0.14018 rpy=1.5708 -1.5708 0, axis 0 0 -1, limit lower=-1.57 upper=1.57 effort=30.0 velocity=10
- added joint z1_gripperStator: type fixed, parent link06, child gripperStator, origin xyz=-0.0056012 -0.029636 0.0706 rpy=-1.5714 -1.5708 0
- added joint z1_jointGripper: type prismatic, parent gripperStator, child gripperMover, origin xyz=-0.0056012 0.02964 0.0706 rpy=0 0 0, axis 0 0 1, limit lower=-0.03 upper=0 effort=30 velocity=10
- added joint z1_shoulder: type revolute, parent link01, child link02, origin xyz=0 0.028 0.0563 rpy=1.5708 0 -3.1416, axis 0 0 -1, limit lower=-1.57 upper=1.57 effort=60.0 velocity=10
- added joint z1_waist: type revolute, parent link00, child link01, origin xyz=0 0 0.0533 rpy=0 0 -3.1416, axis 0 0 1, limit lower=-2.35 upper=2.35 effort=30 velocity=10
- added joint z1_wrist_angle: type revolute, parent link03, child link04, origin xyz=0.0577 0.042 -0.0275 rpy=-1.5708 0 -1.5708, axis 0 0 1, limit lower=-2.35 upper=2.35 effort=30.0 velocity=10
- added joint z1_wrist_rotate: type revolute, parent link05, child link06, origin xyz=0.0825 -0.0010782 -0.023822 rpy=-1.5708 0 -1.5708, axis 0 0 -1, limit lower=-2.35 upper=2.35 effort=30.0 velocity=10

Commit message: Test on Go2D1

File: low-level/resources/robots/go2d1/urdf/go2d1.urdf (robot description, URDF)
Before this commit: robot go2d1_description, 29 links, 28 joints
Links:
- removed link imu_link
- added link FL_calflower; collision cylinder length=0.065 radius=0.011
- added link FL_calflower1; collision cylinder length=0.03 radius=0.0155
- added link FR_calflower; collision cylinder length=0.065 radius=0.011
- added link FR_calflower1; collision cylinder length=0.03 radius=0.0155
- added link Head_lower, mass 0.001; collision sphere radius=0.047
- added link Head_upper, mass 0.001; collision cylinder length=0.09 radius=0.05
- added link RL_calflower; collision cylinder length=0.065 radius=0.011
- added link RL_calflower1; collision cylinder length=0.03 radius=0.0155
- added link RR_calflower; collision cylinder length=0.065 radius=0.011
- added link RR_calflower1; collision cylinder length=0.03 radius=0.0155
- added link imu, mass 0
- added link radar, mass 0
- link FL_calf: geometry collision cylinder length=0.12 radius=0.012; visual mesh filename=../meshes/calf.dae
- link FL_hip: geometry collision cylinder length=0.04 radius=0.046; visual mesh filename=../meshes/hip.dae
- link FL_thigh: geometry collision box size=0.213 0.0245 0.034; visual mesh filename=../meshes/thigh.dae
- link FR_calf: geometry collision cylinder length=0.12 radius=0.013; visual mesh filename=../meshes/calf_mirror.dae
- link FR_hip: geometry collision cylinder length=0.04 radius=0.046; visual mesh filename=../meshes/hip.dae
- link FR_thigh: geometry collision box size=0.213 0.0245 0.034; visual mesh filename=../meshes/thigh_mirror.dae
- link RL_calf: geometry collision cylinder length=0.12 radius=0.013; visual mesh filename=../meshes/calf.dae
- link RL_hip: geometry collision cylinder length=0.04 radius=0.046; visual mesh filename=../meshes/hip.dae
- link RL_thigh: geometry collision box size=0.213 0.0245 0.034; visual mesh filename=../meshes/thigh.dae
- link RR_calf: geometry collision cylinder length=0.12 radius=0.013; visual mesh filename=../meshes/calf_mirror.dae
- link RR_hip: geometry collision cylinder length=0.04 radius=0.046; visual mesh filename=../meshes/hip.dae
- link RR_thigh: geometry collision box size=0.213 0.0245 0.034; visual mesh filename=../meshes/thigh_mirror.dae
- link link00: geometry collision mesh filename=../meshes/d1_Link00.dae; visual mesh filename=../meshes/d1_Link00.dae
- link link01: geometry collision mesh filename=../meshes/d1_Link01.dae; visual mesh filename=../meshes/d1_Link01.dae
- link link02: geometry collision mesh filename=../meshes/d1_Link02.dae; visual mesh filename=../meshes/d1_Link02.dae
- link link03: geometry collision mesh filename=../meshes/d1_Link03.dae; visual mesh filename=../meshes/d1_Link03.dae
- link link04: geometry collision mesh filename=../meshes/d1_Link04.dae; visual mesh filename=../meshes/d1_Link04.dae
- link link05: geometry collision mesh filename=../meshes/d1_Link05.dae; visual mesh filename=../meshes/d1_Link05.dae
- link link06: geometry collision mesh filename=../meshes/d1_Link06.dae; visual mesh filename=../meshes/d1_Link06.dae
- link trunk: mass 25 -> 6.921; geometry collision box size=0.3762 0.0935 0.114; visual mesh filename=../meshes/trunk.dae
Joints:
- removed joint FL_foot_fixed
- removed joint FR_foot_fixed
- removed joint RL_foot_fixed
- removed joint RR_foot_fixed
- added joint FL_calflower1_joint: type fixed, parent FL_calflower, child FL_calflower1, origin xyz=-0.01 0 -0.04 rpy=0 0.48 0, axis 0 0 0
- added joint FL_calflower_joint: type fixed, parent FL_calf, child FL_calflower, origin xyz=0.020 0 -0.148 rpy=0 0.05 0, axis 0 0 0
- added joint FL_foot_joint: type fixed, parent FL_calf, child FL_foot, origin xyz=0 0 -0.213 rpy=0 0 0, axis 0 0 0
- added joint FR_calflower1_joint: type fixed, parent FR_calflower, child FR_calflower1, origin xyz=-0.01 0 -0.04 rpy=0 0.48 0, axis 0 0 0
- added joint FR_calflower_joint: type fixed, parent FR_calf, child FR_calflower, origin xyz=0.020 0 -0.148 rpy=0 0.05 0, axis 0 0 0
- added joint FR_foot_joint: type fixed, parent FR_calf, child FR_foot, origin xyz=0 0 -0.213 rpy=0 0 0, axis 0 0 0
- added joint Head_lower_joint: type fixed, parent Head_upper, child Head_lower, origin xyz=0.008 0 -0.07 rpy=0 0 0, axis 0 0 0
- added joint Head_upper_joint: type fixed, parent base, child Head_upper, origin xyz=0.285 0 0.01 rpy=0 0 0, axis 0 0 0
- added joint RL_calflower1_joint: type fixed, parent RL_calflower, child RL_calflower1, origin xyz=-0.01 0 -0.04 rpy=0 0.48 0, axis 0 0 0
- added joint RL_calflower_joint: type fixed, parent RL_calf, child RL_calflower, origin xyz=0.020 0 -0.148 rpy=0 0.05 0, axis 0 0 0
- added joint RL_foot_joint: type fixed, parent RL_calf, child RL_foot, origin xyz=0 0 -0.213 rpy=0 0 0, axis 0 0 0
- added joint RR_calflower1_joint: type fixed, parent RR_calflower, child RR_calflower1, origin xyz=-0.01 0 -0.04 rpy=0 0.48 0, axis 0 0 0
- added joint RR_calflower_joint: type fixed, parent RR_calf, child RR_calflower, origin xyz=0.020 0 -0.148 rpy=0 0.05 0, axis 0 0 0
- added joint RR_foot_joint: type fixed, parent RR_calf, child RR_foot, origin xyz=0 0 -0.213 rpy=0 0 0, axis 0 0 0
- added joint radar_joint: type fixed, parent base, child radar, origin xyz=0.28945 0 -0.046825 rpy=0 2.8782 0, axis 0 0 0
- joint FL_hip_joint: parent trunk -> base
- joint FR_hip_joint: parent trunk -> base
- joint RL_hip_joint: parent trunk -> base
- joint RR_hip_joint: parent trunk -> base
- joint base_static_joint: origin xyz=0 0 0.05 rpy=0 0 0 -> xyz=0 0 0.06 rpy=0 0 0
- joint ee_gripper: origin xyz=0.135 0 0 rpy=0 0 0 -> xyz=0.01 0.02 0.02 rpy=0 0 0
- joint imu_joint: axis (none) -> 0 0 0; child imu_link -> imu; origin xyz=0 0 0 rpy=0 0 0 -> xyz=-0.02557 0 0.04232 rpy=0 0 0; parent trunk -> base
- joint z1_elbow: limit lower=-1.57 upper=1.57 effort=30.0 velocity=10 -> lower=-1.57 upper=1.57 effort=10 velocity=3
- joint z1_forearm_roll: limit lower=-1.57 upper=1.57 effort=30.0 velocity=10 -> lower=-1.57 upper=1.57 effort=10 velocity=3
- joint z1_jointGripper: limit lower=-0.03 upper=0 effort=30 velocity=10 -> lower=-0.03 upper=0.0 effort=30.0 velocity=0.05; origin xyz=-0.0056012 0.02964 0.0706 rpy=0 0 0 -> xyz=-0.0056388 0.02964 0.0706 rpy=1.5702 -1.5708 0; parent gripperStator -> link06
- joint z1_shoulder: limit lower=-1.57 upper=1.57 effort=60.0 velocity=10 -> lower=-1.57 upper=1.57 effort=20 velocity=3
- joint z1_waist: limit lower=-2.35 upper=2.35 effort=30 velocity=10 -> lower=-2.35 upper=2.35 effort=10 velocity=3
- joint z1_wrist_angle: limit lower=-2.35 upper=2.35 effort=30.0 velocity=10 -> lower=-2.35 upper=2.35 effort=10 velocity=3
- joint z1_wrist_rotate: limit lower=-2.35 upper=2.35 effort=30.0 velocity=10 -> lower=-2.35 upper=2.35 effort=10 velocity=3

Commit message: Follow latest update 7243de4 from upstream and personal modify

File: low-level/resources/robots/go2d1/urdf/go2d1.urdf (robot description, URDF)
Before this commit: robot b1z1_description, 40 links, 39 joints
Links:
- removed link Head_lower
- removed link Head_upper
Joints:
- removed joint Head_lower_joint
- removed joint Head_upper_joint
- joint FL_hip_joint: parent base -> trunk
- joint FR_hip_joint: parent base -> trunk
- joint RL_hip_joint: parent base -> trunk
- joint RR_hip_joint: parent base -> trunk
- joint imu_joint: parent base -> trunk
- joint radar_joint: parent base -> trunk

Commit message: prepare go2d1 high-level

File: low-level/resources/robots/go2d1/urdf/go2d1.urdf (robot description, URDF)
Before this commit: robot b1z1_description, 38 links, 37 joints
Joints:
- joint z1_jointGripper: limit lower=-0.03 upper=0.0 effort=30.0 velocity=0.05 -> lower=-0.03 upper=0.0 effort=5.0 velocity=1
