Commit message: improve low-level on go2; check high-level problems on coordinates between arm and base

File: high-level/data/asset/go2d1/urdf/go2d1.urdf (robot description, URDF)
Before this commit: robot b1z1_description, 38 links, 37 joints
Joints:
- joint z1_jointGripper: limit lower=-0.03 upper=0.0 effort=5.0 velocity=1 -> lower=-0.03 upper=0.0 effort=10.0 velocity=3
